Commit message: Update to make lidar aligned with chassis

File: Where-Am-I/src/my_robot/urdf/my_robot.xacro (robot description, xacro)
@@ -169,5 +169,5 @@
 		</collision>
 		<visual name='lidar_visual'>
-			<origin xyz="0.20 0 0" rpy=" 0 0 0"/>
+			<origin xyz="0.0 0 0" rpy=" 0 0 0"/>
 			<geometry>
 				<mesh filename="package://my_robot/meshes/hokuyo.dae"/>
@@ -176,5 +176,5 @@
 	</link>
 	<joint type="fixed" name="hokuyo_joint">
-		<origin xyz="0.15 0 0.1" rpy="0 0 0"/>
+		<origin xyz="0.15 0 0.05" rpy="0 0 0"/>
 		<child link="hokuyo"/>
 		<parent link="chassis"/>
